File: OCP-1/OCP-1.sch (KiCad schematic (older format))
At the start: 8 parts

Commit message: изменен ac-dc и дублирующий контроллер на esp32
Parts:
- removed G1: AC-DC-преобразователь_LS05-15B05SS, symbol elements_2020:AC-DC-преобразователь_LS05-15B05SS
- added C10, C6, C8, C9: Конденсатор_керамический, N_RLC:Конденсатор_SMD_0805, symbol elements:Конденсатор_керамический
- added C7: Конденсатор_электролитический, symbol elements:Конденсатор_электролитический
- added G1: AC-DC-преобразователь_AMEOF3-5SJZ, symbol elements_2020:AC-DC-преобразователь_AMEOF3-5SJZ
- added G2: стабилизатор_нерегулируемый_LM1117S33, N_VD_HL:Транзистор_NPN_SOT223, symbol elements:стабилизатор_нерегулируемый_LM1117S33
- added HL1: Светодиод_сдвоенный_KPB-3025SURKCGKC, N_VD_HL:Светодиод_SMD_m3025, symbol elements_2020:Светодиод_сдвоенный_KPB-3025SURKCGKC
- added L1: Чип-индуктивность, N_RLC:Чип-индуктивность_SMD_1210, symbol elements:Чип-индуктивность
- added R1: Резистор_0,25Вт, N_RLC:Резистор_SMD_1206-0,25_Вт_pnp, symbol elements:Резистор_0,25Вт
- added X1: Клеммник_х2, N_X:Клеммник_х2_шаг5, symbol elements:Клеммник_х2
- added XFU1, XFU2: Держатель_предохранителя_KLS5-266, N_X:Держатель_5х20, symbol elements_2020:Держатель_предохранителя_KLS5-266
Connections:
- net labels added: 0V, 3V3, 5V
- wire segments 27 -> 66
Other:
- note added: "MC"
- moved on the sheet: C1, C2, C3, C4, VD1

Commit message: теперь это альтиметр со звуковым оповещением
Parts:
- removed C1, C2, C4, C7: Конденсатор_электролитический, symbol elements:Конденсатор_электролитический
- removed C10, C3, C6, C8, C9: Конденсатор_керамический, N_RLC:Конденсатор_SMD_0805, symbol elements:Конденсатор_керамический
- removed C5: Конденсатор_керамический, N_RLC:Конденсатор_SMD_2220, symbol elements:Конденсатор_керамический
- removed G1: AC-DC-преобразователь_AMEOF3-5SJZ, symbol elements_2020:AC-DC-преобразователь_AMEOF3-5SJZ
- removed G2: стабилизатор_нерегулируемый_LM1117S33, N_VD_HL:Транзистор_NPN_SOT223, symbol elements:стабилизатор_нерегулируемый_LM1117S33
- removed HL1: Светодиод_сдвоенный_KPB-3025SURKCGKC, N_VD_HL:Светодиод_SMD_m3025, symbol elements_2020:Светодиод_сдвоенный_KPB-3025SURKCGKC
- removed L1: Чип-индуктивность, N_RLC:Чип-индуктивность_SMD_1210, symbol elements:Чип-индуктивность
- removed R1: Резистор_0,25Вт, N_RLC:Резистор_SMD_1206-0,25_Вт_pnp, symbol elements:Резистор_0,25Вт
- removed RK1: Термистор, symbol elements:Термистор
- removed VD1: Диод_шоттки_SK16, N_VD_HL:Диод_SMB_pnp, symbol elements_2020:Диод_шоттки_SK16
- removed X1: Клеммник_х2, N_X:Клеммник_х2_шаг5, symbol elements:Клеммник_х2
- removed XFU1, XFU2: Держатель_предохранителя_KLS5-266, N_X:Держатель_5х20, symbol elements_2020:Держатель_предохранителя_KLS5-266
- added DA1, DA2: ОУ_LMx58, N_DD:SO-8, symbol elements:ОУ_LMx58
- added DD1: 1986ВЕ92QL, N_DD:Микросхема_1986ВЕ92QL, symbol elements:1986ВЕ92QL
- added DD2: BMP280, N_DD:BMP280, symbol elements_2020:BMP280
- added R1, R2, R3, R4, R5, R6, R7, R8: Резистор_0,065Вт, N_RLC:Резистор_SMD_0603_0,065_Вт, symbol elements:Резистор_0,065Вт
- added VT1, VT2: Транзистор_полевой_P-канал(IRLML2246TRPBF), N_VD_HL:Транзистор_IRLML6344TR_SOT-23, symbol elements:Транзистор_полевой_P-канал(IRLML2246TRPBF)
- added VT3: Транзистор_полевой_N-IRLML6344TR, N_VD_HL:Транзистор_IRLML6344TR_SOT-23, symbol elements:Транзистор_полевой_N-IRLML6344TR
Connections:
- new net: R1.1, R2.2, VT1.1
- new net: R5.1, R6.1, R7.1, R8.1
- new net: R5.2, R6.2, R7.2, R8.2
- new net: R3.2, R4.1, VT2.1
- new net 4V2.DIRECT: DA1.1, R4.2
- new net 4V2.OUT: DA1.3, VT2.3
- new net 4V2.REF: DA1.2
- new net 5V.IN: VT1.3
- new net 5V.LINE: DA1.8 (VCC+), R2.1, R3.1, VT1.2, VT2.2
- new net GND: DA1.4 (-VCC), R1.2
Other:
- note added: "защита от \nпереполюсовки"
- note removed: "MC"

Commit message: схема заряда аккумулятора и требования к питанию периферии
Parts:
- added DD3: LIS3DH, N_DD:акселерометр_LIS3DH, symbol elements:LIS3DH
- added G1: ИОП_LM4040BIM3-2.5_NOPB, N_VD_HL:Транзистор_IRLML6344TR_SOT-23, symbol elements_2020:ИОП_LM4040BIM3-2.5_NOPB
- added HL1, HL2: Светодиод_сдвоенный_KPB-3025SURKCGKC, N_VD_HL:Светодиод_SMD_m3025, symbol elements_2020:Светодиод_сдвоенный_KPB-3025SURKCGKC
- added K1, K2, K3, K4: Кнопка_KLS7-TS5401-1.35-250-T, N_X:Кнопка_KLS7-TS5401, symbol elements_2020:Кнопка_KLS7-TS5401-1.35-250-T
- added R10, R11, R12, R13, R14, R15, R16, R17, R18, R19, R9: Резистор_0,065Вт, N_RLC:Резистор_SMD_0603_0,065_Вт, symbol elements:Резистор_0,065Вт
- added VT4: Транзистор_полевой_P-канал(IRLML2246TRPBF), N_VD_HL:Транзистор_IRLML6344TR_SOT-23, symbol elements:Транзистор_полевой_P-канал(IRLML2246TRPBF)
- added X1: Клеммник_х2, N_X:Клеммник_х2_шаг2.54, symbol elements:Клеммник_х2
Connections:
- net 5V.LINE: now also DA2.8 (VCC+), R10.1, R9.1, VT4.2; no longer R3.1, VT2.2
- net GND: now also DA2.4 (-VCC), G1.2, R13.2, R16.2, R19.2, X1.2
- net DIFF.AMP: now reaches DA1.5
- net DIFF.AMP: now also DA2.1, R17.1
- net 1V5.REF: now reaches DA1.6
- net 1V5.REF: now also R18.2, R19.1
- net CUR.DIRECT: now reaches DA1.7
- net CUR.DIRECT: now also R11.2
- net at DA2.2: now also R14.1, R17.2
- net at DA2.3: now also R15.1, R16.1
- net CUR.OUT: now reaches DA2.5
- net CUR.OUT: now also R3.1, R5.2, R6.2, R7.2, R8.2, VT2.2
- net REP.SENS-: now reaches DA2.6
- net REP.SENS-: now also DA2.7, R14.2
- net CUR.SENS: now reaches R5.1, R6.1, R7.1, R8.1
- net CUR.SENS: now also R15.2, VT4.3
- net 4V2.OUT renamed 2V5.OUT
- net 2V5.OUT: now also R12.2, R13.1; no longer VT2.3
- net 4V2.REF renamed 2V5.REF
- net 2V5.REF: now also G1.1, R18.1, R9.2
- new net: R10.2, R11.1, VT4.1
- new net 4V1.OUT: R12.1, VT2.3, X1.1
Other:
- note added: "0,5А/0,125В\n0,3А/0,075В\n0,3А/0,075В"
- note added: "1,5В->0,3А"
- note added: "2,46В\n1,498В\n1,506В"
- note added: "4,76В\n5,238В\n4,286В"
- note added: "4,875В\n5,425В\n4,425В"
- note added: "5В,\n5,5В\n4,5В"
- note added: "Udiff = Umid - (Umin - Umid)*R4/R3"
- note added: "Питание:\nмикроконтроллер - 3,3В\nакселерометр - 2,5В\nальтиметр - 1,8В"
- note added: "кнопка питания\nкнопка вверх\nкнопка вниз\nкнопка назад"
- note added: "светодиод запись/ожидание\nсветодиод заряд/глубокий разряд"
- note added: "стабилизатор \nнапряжения (4,1…4,2)В"
- note added: "стабилизатор\nтока max 0,3А"
- moved on the sheet: DA1, DD1, DD2, R1, R2, R3, R4, R5, R6, R7, R8, VT1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
