File: OCP-1/OCP-1.sch (KiCad schematic (older format))
At the start: 50 parts, among them K1 Кнопка_KLS7-TS5401-1.35-250-T, K2 Кнопка_KLS7-TS5401-1.35-250-T, K3 Кнопка_KLS7-TS5401-1.35-250-T, K4 Кнопка_KLS7-TS5401-1.35-250-T, X1 Клеммник_х2

Commit message: добавлена схема включения и расположение индикаторов
Parts:
- removed C7: Конденсатор_керамический, N_RLC:Конденсатор_SMD_IEC_0805, symbol elements:Конденсатор_керамический
- removed G3: LDO_TPS76325DBVR, N_G:Преобразователь_LM2703_SOT-23-5, symbol elements_2020:LDO_TPS76325DBVR
- removed K1, K3, K4: Кнопка_KLS7-TS5401-1.35-250-T, N_X:Кнопка_KLS7-TS5401, symbol elements_2020:Кнопка_KLS7-TS5401-1.35-250-T
- added HL3, HL4, HL5, HL6: Индикатор_7сегм_TOS-F2101AMG, N_VD_HL:LED-7SEGM-10x6,9, symbol elements_2020:Индикатор_7сегм_TOS-F2101AMG
- added K1, K3, K4, K5: кнопка, N_X:Кнопка_FSMSM, symbol elements:кнопка
- added R24, R25, R26, R27: Резистор_0,065Вт, N_RLC:Резистор_SMD_0603_0,065_Вт, symbol elements:Резистор_0,065Вт
- added VD1: Диоды_шоттки_BAR43CFILM, N_VD_HL:Транзистор_IRLML6344TR_SOT-23, symbol elements_2020:Диоды_шоттки_BAR43CFILM
- added VT5: Транзистор_полевой_P-канал(IRLML2246TRPBF), N_VD_HL:Транзистор_IRLML6344TR_SOT-23, symbol elements:Транзистор_полевой_P-канал(IRLML2246TRPBF)
- added VT6: Транзистор_полевой_N-канальный_КП526А9, MOTOR_VD_VT_HL:Корпус_КТ-46, symbol elements_2020:Транзистор_полевой_N-канальный_КП526А9
- G1: footprint N_VD_HL:Транзистор_IRLML6344TR_SOT-23 -> MOTOR_VD_VT_HL:Корпус_КТ-46; INFO - -> 2V5
- R12: Номинал 20 кОм -> 39 кОм
- R13: Номинал 30 кОм -> 22 кОм
- R19: Номинал 15 кОм -> 10 кОм
Connections:
- net 1V5.REF: no longer R18.2, R19.1
- net 2V5: now also G1.1, R9.2, R26.1
- net 4V1.OUT: now also R18.2, VT5.2; no longer R20.1, VT3.2
- net GND: now also K2.2, K2.4, K1.1, K3.1, K4.1, K5.1, R27.2, VT6.2
- net RES: now reaches K2.1
- net RES: now also K2.3
- net 2V5.FB1 renamed 1V5.FB1
- removed net 2V5.REF: DA1.2, G1.1, R18.1, R9.2
- new net: R20.1, VT3.2, VT5.3
- new net: R18.1, VD1.1, VD1.2, VT5.1, VT6.3
- new net: R19.1, R24.2, VT6.1
- new net 1V225.REF: DA1.2
- new net 1V25.REF: R26.2, R27.1
- new net B-BACK: K4.2
- new net B-DOWN: K3.2
- new net B-PWR: K5.2, R25.2, VD1.3
- new net B-UP: K1.2
- new net SELF-TURN: R24.1
- new net SENS-B-PWR: R25.1
- no-connect marks 5 -> 4
Other:
- note added: "10 мА MAX"
- note added: "Питание:\nмикроконтроллер - 3,0...3,2В\nакселерометр - 2,5В (3,0...3,2В)\nальтиметр - 1,8В"
- note added: "разрешение включения"
- note removed: "Питание:\nмикроконтроллер - 3,0...3,2В\nакселерометр - 2,5В\nальтиметр - 1,8В"
- moved on the sheet: C3, C4, C5, C6, DA1, DA3, DD1, DD2, DD3, G1, G4, K2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

Commit message: заготовка usb-type-c
Parts:
- added XS1: UBS-tupe-C-105450-0101&упрощенная, symbol elements_2020:UBS-tupe-C-105450-0101&упрощенная
Changed lines of the file:
@@
 EESchema Schematic File Version 4
 LIBS:OCP-1-cache
-EELAYER 30 0
+EELAYER 29 0
 EELAYER END
 $Descr A1 33110 23386
@@
 	1    0    0    -1
 $EndComp
+$Comp
+L elements_2020:UBS-tupe-C-105450-0101&упрощенная XS1
+U 1 1 617F4717
+P 5050 12500
+F 0 "XS1" H 5475 12900 138 0000 L CNN
+F 1 "UBS-tupe-C-105450-0101&упрощенная" H 5250 13200 50  0001 C CNN
+F 2 "" H 5050 12500 50  0001 C CNN
+F 3 "" H 5050 12500 50  0001 C CNN
+F 4 "https://www.chipdip.ru/product/105450-0101-molex" H 5050 13100 50  0001 C CNN "LINK"
+	1    5050 12500
+	1    0    0    -1
+$EndComp

Commit message: определена схема индикаторов, динамика, не исправлены резисторы питания
Parts:
- added C7: Конденсатор_керамический, N_RLC:Конденсатор_SMD_IEC_0805, symbol elements:Конденсатор_керамический
- added R28, R29, R30, R31, R32, R33, R34, R35, R36, R37, R38, R39, R40, R41, R42, R43, R44, R45, R46, R47, R50, R51: Резистор_0,065Вт, N_RLC:Резистор_SMD_0603_0,065_Вт, symbol elements:Резистор_0,065Вт
- added VT13, VT14, VT7, VT8, VT9: Транзистор_полевой_N-канальный_КП526А9, MOTOR_VD_VT_HL:Корпус_КТ-46, symbol elements_2020:Транзистор_полевой_N-канальный_КП526А9
- added XP1: СНП346-6ВП_(отладочная), MOTOR_X:Вилка_СНП346_6, symbol MOTOR:СНП346-6ВП_(отладочная)
- added XТ1: Клеммник_х2, N_X:Клеммник_х2_шаг2.54, symbol elements:Клеммник_х2
- XS1: value UBS-tupe-C-105450-0101&упрощенная -> UBS-type-C-105450-0101&упрощенная; footprint (none) -> N_X:usb-type-c; symbol elements_2020:UBS-tupe-C-105450-0101&упрощенная -> elements_2020:UBS-type-C-105450-0101&упрощенная
Connections:
- net 1V5.FB1 is gone; now on net BAT.1V5.FB1: DA1.3, R12.2, R13.1
- net 3V1: now also DD1.1 (DUcc), DD1.12 (DUcc), DD1.13 (BUcc), DD1.24 (AUcc1), DD1.28 (AUcc), DD1.38 (DUcc), DD1.48 (DUcc)
- net 5V.IN: now also XS1.A4 (VBUS), XS1.A9 (VBUS), XS1.B4 (VBUS), XS1.B9 (VBUS)
- net B-BACK: now also R34.2; no longer K4.2
- net B-DOWN: now also R30.2; no longer K3.2
- net B-PWR: now also R31.2; no longer K5.2
- net B-UP: now also R29.2; no longer K1.2
- net DIFF.AMP: now also DD1.29 (PD7)
- net GND: now also DD1.11 (DGND), DD1.23 (AGND1), DD1.27 (AGND), DD1.39 (DGND), DD1.49 (DGND), DD1.64 (DGND), XS1.A1 (GND), XS1.A12 (GND), XS1.B1 (GND), XS1.B12 (GND), R38.2, R39.2, R47.2, R50.2, R51.2, VT13.2, VT14.2, VT7.2, VT8.2, VT9.2
- net RES: now also DD1.18 (RESET)
- net USBD-: now reaches DD1.10 (DN)
- net USBD-: now also XS1.A6 (D+), XS1.B6 (D+)
- net TMS: now reaches DD1.31 (PD0(JB_TMS)/RX101)
- net TCK: now reaches DD1.32 (PD1(JB_TCK)/TX101)
- net BAT.1V5.FB1: now reaches DD1.36 (PD6)
- net SDA: now reaches DD1.41 (PC1)
- net SCL: now reaches DD1.42 (PC0)
- net T3C4: now reaches DD1.52 (PB7)
- net T3C4: now also R46.2
- net DP: now reaches DD1.56 (PA7)
- net DP: now also R43.2
- net G: now reaches DD1.57 (PA6)
- net G: now also R42.2
- net F: now reaches DD1.58 (PA5)
- net F: now also R41.2
- net E: now reaches DD1.59 (PA4)
- net E: now also R40.2
- net D: now reaches DD1.60 (PA3)
- net D: now also R37.2
- net C: now reaches DD1.61 (PA2)
- net C: now also R36.2
- net B: now reaches DD1.62 (PA1)
- net B: now also R35.2
- net A: now reaches DD1.63 (PA0)
- net A: now also R28.2
- net USBD+: now reaches DD1.9 (DP)
- net USBD+: now also XS1.A7 (D-), XS1.B7 (D-)
- net V.BATT: now reaches R20.1, VT3.2, VT5.3
- net V.BATT: now also XТ1.1
- net HL.E: now reaches HL3.1 (E)
- net HL.E: now also HL4.1 (E), HL5.1 (E), HL6.1 (E), R40.1
- net HL.G: now reaches HL3.10 (G)
- net HL.G: now also HL4.10 (G), HL5.10 (G), HL6.10 (G), R42.1
- net HL.D: now reaches HL3.2 (D)
- net HL.D: now also HL4.2 (D), HL5.2 (D), HL6.2 (D), R37.1
- net HL1.C: now reaches HL3.3 (~COM)
- net HL1.C: now also HL3.8 (~COM), VT7.3
- net HL.C: now reaches HL3.4 (C)
- net HL.C: now also HL4.4 (C), HL5.4 (C), HL6.4 (C), R36.1
- net HL.DP: now reaches HL3.5 (DP)
- net HL.DP: now also HL4.5 (DP), HL5.5 (DP), HL6.5 (DP), R43.1
- net HL.B: now reaches HL3.6 (B)
- net HL.B: now also HL4.6 (B), HL5.6 (B), HL6.6 (B), R35.1
- net HL.A: now reaches HL3.7 (A)
- net HL.A: now also HL4.7 (A), HL5.7 (A), HL6.7 (A), R28.1
- net HL.F: now reaches HL3.9 (F)
- net HL.F: now also HL4.9 (F), HL5.9 (F), HL6.9 (F), R41.1
- net HL2.C: now reaches HL4.3 (~COM)
- net HL2.C: now also HL4.8 (~COM), VT8.3
- net HL3.C: now reaches HL5.3 (~COM)
- net HL3.C: now also HL5.8 (~COM), VT13.3
- net HL4.C: now reaches HL6.3 (~COM)
- net HL4.C: now also HL6.8 (~COM), VT14.3
- new net: K5.2, R31.1
- new net: K4.2, R34.1
- new net: K1.2, R29.1
- new net: K3.2, R30.1
- new net: R32.1, R38.1, VT7.1
- new net: R44.1, R50.1, VT13.1
- new net: R45.1, R51.1, VT14.1
- new net: R33.1, R39.1, VT8.1
- new net: R46.1, R47.1, VT9.1
- new net: C7.2, VT9.3
- new net: C7.1, XТ1.2
- new net HL1: R32.2
- new net HL2: R33.2
- new net HL3: R44.2
- new net HL4: R45.2
- no-connect marks 4 -> 9
Other:
- note added: "добавить ограничтельные резисторы"
- moved on the sheet: DD1, DD2, DD3, HL1, HL2, HL3, HL4, HL5, HL6, K1, K2, K3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
